File: react_schematics/react_schematics.kicad_sch (KiCad schematic)
At the start: 24 parts, among them J1 Input Jack, J2 Input Jack, SW1 221ADA10, U1 MPM3610, U2 DS3231M, U3 MAX485E, U4 ICM-42688-P

Commit message: new schematics
Parts:
- removed C1, C2: 22uF, react_schematics:0805-NO, symbol react_schematics-eagle-import:CAP_CERAMIC0805-NOOUTLINE
- removed J1, J2: Input Jack, symbol Connector:RJ45_Shielded
- removed R1, R2: 100K, react_schematics:0603-NO, symbol react_schematics-eagle-import:RESISTOR_0603_NOOUT
- removed R3: 18.7K, react_schematics:0603-NO, symbol react_schematics-eagle-import:RESISTOR_0603_NOOUT
- removed U1: MPM3610, react_schematics:MPM3610, symbol react_schematics-eagle-import:MPM3610
Connections:
- net +5V is gone; now on net 5V PPWR: C7.2, C8.2, U3.8 (VCC)
- net 5V PPWR: now also A1.40 (VBUS)
- net ABORT_SIG: now also A1.34 (GPIO28_ADC2); no longer A1.32 (GPIO27_ADC1)
- net GND: now also U2.10 (GND), U2.11 (GND), U2.12 (GND), U2.13 (GND), U2.5 (GND), U2.6 (GND), U2.7 (GND), U2.8 (GND), U2.9 (GND)
- net RS485_RX: now reaches A1.2 (GPIO1), U3.1 (RO)
- net RS485_RX: now also U3.2 (~{RE}), U3.3 (DE)
- net RS485_TX: now reaches A1.1 (GPIO0), U3.4 (DI)
- new net RS485_RTS: A1.4 (GPIO2)
- no-connect marks 23 -> 19
Other:
- added sheet Power and Connectors (power_and_connectors.kicad_sch)
- moved on the sheet: C5, C7, C8, R4, U2, U3

Commit message: new sch changes
Connections:
- net RS485_RTS: now also U3.2 (~{RE}), U3.3 (DE)
- net RS485_RX: no longer U3.2 (~{RE}), U3.3 (DE)
- net TERM_SIG: now reaches A1.31 (GPIO26_ADC0)
- net ABORT_SIG_OUT: now reaches A1.32 (GPIO27_ADC1)
- net ABORT_SIG renamed ABORT_SIG_IN
- no-connect marks 19 -> 22
Other:
- added sheet Host Console (host_console.kicad_sch)
- sheet Power and Connectors ports: added ABORT_SIG_IN, ABORT_SIG_OUT, TERM_SIG; removed ABORT_SIG
Changed lines of the file:
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@@
 	)
 	(no_connect
-		(at 99.06 76.2)
+		(at 53.34 58.42)
+	)
+	(no_connect
+		(at 53.34 81.28)
 	)
 	(no_connect
@@
 	)
 	(no_connect
+		(at 53.34 38.1)
+	)
+	(no_connect
 		(at 99.06 68.58)
 	)
 	(no_connect
-		(at 53.34 73.66)
+		(at 53.34 53.34)
 	)
 	(no_connect
-		(at 166.37 151.13)
+		(at 53.34 40.64)
+	)
+	(no_connect
+		(at 53.34 73.66)
 	)
 	(no_connect
-		(at 53.34 80.01)
+		(at 166.37 151.13)
 	)
 	(no_connect
@@
 	)
 	(no_connect
+		(at 53.34 55.88)
+	)
+	(no_connect
 		(at 166.37 153.67)
 	)
@@
 	)
 	(no_connect
-		(at 99.06 73.66)
-	)
-	(no_connect
 		(at 99.06 60.96)
 	)
@@
 	(wire
 		(pts
+			(xy 217.17 63.5) (xy 232.41 63.5)
+		)
+		(stroke
+			(width 0)
+			(type default)
+		)
+	)
+	(wire
+		(pts
 			(xy 41.91 63.5) (xy 53.34 63.5)
 		)
@@
 	(wire
 		(pts
+			(xy 99.06 76.2) (xy 101.6 76.2)
+		)
+		(stroke
+			(width 0)
+			(type default)
+		)
+	)
+	(wire
+		(pts
 			(xy 190.5 102.87) (xy 190.5 109.22)
 		)
@@
 	(wire
 		(pts
+			(xy 99.06 73.66) (xy 101.6 73.66)
+		)
+		(stroke
+			(width 0)
+			(type default)
+		)
+	)
+	(wire
+		(pts
 			(xy 55.88 127) (xy 58.42 127)
 		)
@@
 	(wire
 		(pts
+			(xy 217.17 60.96) (xy 232.41 60.96)
+		)
+		(stroke
+			(width 0)
+			(type default)
+		)
+	)
+	(wire
+		(pts
 			(xy 45.72 102.87) (xy 45.72 106.68)
 		)
@@
 	(wire
 		(pts
-			(xy 220.98 53.34) (xy 232.41 53.34)
+			(xy 217.17 58.42) (xy 232.41 58.42)
 		)
 		(stroke
@@
 	(wire
 		(pts
-			(xy 220.98 48.26) (xy 232.41 48.26)
+			(xy 218.44 48.26) (xy 232.41 48.26)
 		)
 		(stroke
@@
 	(wire
 		(pts
-			(xy 220.98 45.72) (xy 232.41 45.72)
+			(xy 218.44 45.72) (xy 232.41 45.72)
 		)
 		(stroke
@@
 	(wire
 		(pts
-			(xy 220.98 55.88) (xy 232.41 55.88)
+			(xy 218.44 53.34) (xy 232.41 53.34)
 		)
 		(stroke
@@
 	(wire
 		(pts
-			(xy 220.98 50.8) (xy 232.41 50.8)
+			(xy 218.44 50.8) (xy 232.41 50.8)
 		)
 		(stroke
@@
 		)
 	)
+	(label "ABORT_SIG_OUT"
+		(at 217.17 60.96 0)
+		(effects
+			(font
+				(size 1.27 1.27)
+			)
+			(justify left bottom)
+		)
+	)
+	(label "TERM_SIG"
+		(at 101.6 73.66 0)
+		(effects
+			(font
+				(size 1.27 1.27)
+			)
+			(justify left bottom)
+		)
+	)
 	(label "BCD_FOURS"
 		(at 41.91 63.5 0)
@@
 	)
 	(label "GUN_SENSE"
-		(at 220.98 50.8 0)
+		(at 218.44 50.8 0)
 		(effects
 			(font
@@
 	)
 	(label "RS485_B"
-		(at 220.98 48.26 0)
+		(at 218.44 48.26 0)
 		(effects
 			(font
@@
 		)
 	)
-	(label "RS485_RX"
+	(label "RS485_RTS"
 		(at 58.42 127 0)
 		(effects
@@
 		)
 	)
+	(label "ABORT_SIG_OUT"
+		(at 101.6 76.2 0)
+		(effects
+			(font
+				(size 1.27 1.27)
+			)
+			(justify left bottom)
+		)
+	)
 	(label "BCD_TWOS"
 		(at 41.91 66.04 0)
@@
 	)
 	(label "RS485_A"
-		(at 220.98 45.72 0)
+		(at 218.44 45.72 0)
 		(effects
 			(font
@@
 		)
 	)
+	(label "TERM_SIG"
+		(at 217.17 63.5 0)
+		(effects
+			(font
+				(size 1.27 1.27)
+			)
+			(justify left bottom)
+		)
+	)
 	(label "BCD_FOURS"
 		(at 35.56 163.83 0)
@@
 		)
 	)
-	(label "ABORT_SIG"
+	(label "ABORT_SIG_IN"
 		(at 101.6 78.74 0)
 		(effects
@@
 		)
 	)
-	(label "ABORT_SIG"
-		(at 220.98 53.34 0)
+	(label "ABORT_SIG_IN"
+		(at 217.17 58.42 0)
 		(effects
 			(font
@@
 	)
 	(label "FS_ALERT"
-		(at 220.98 55.88 0)
+		(at 218.44 53.34 0)
 		(effects
 			(font
@@
 	)
 	(sheet
+		(at 232.41 109.22)
+		(size 33.02 36.83)
+		(exclude_from_sim no)
+		(in_bom yes)
+		(on_board yes)
+		(dnp no)
+		(fields_autoplaced yes)
+		(stroke
+			(width 0.1524)
+			(type solid)
+		)
+		(fill
+			(color 0 0 0 0.0000)
+		)
+		(property "Sheetname" "Host Console"
+			(at 232.41 108.5084 0)
+			(effects
+				(font
+					(size 1.27 1.27)
+				)
+				(justify left bottom)
+			)
+		)
+		(property "Sheetfile" "host_console.kicad_sch"
+			(at 232.41 146.6346 0)
+			(effects
+				(font
+					(size 1.27 1.27)
+				)
+				(justify left top)
+			)
+		)
+		(instances
+			(project "react_schematics"
+				(path "/097a7a0e-941c-41ac-8d8a-2cc7e0c1dbea"
+					(page "3")
+				)
+			)
+		)
+	)
+	(sheet
 		(at 232.41 40.64)
 		(size 46.99 40.64)
@@
 			)
 		)
-		(pin "ABORT_SIG" bidirectional
+		(pin "FS_ALERT" bidirectional
 			(at 232.41 53.34 180)
 			(effects
@@
 			)
 		)
-		(pin "FS_ALERT" bidirectional
-			(at 232.41 55.88 180)
+		(pin "ABORT_SIG_IN" output
+			(at 232.41 58.42 180)
+			(effects
+				(font
+					(size 1.27 1.27)
+				)
+				(justify left)
+			)
+		)
+		(pin "ABORT_SIG_OUT" output
+			(at 232.41 60.96 180)
+			(effects
+				(font
+					(size 1.27 1.27)
+				)
+				(justify left)
+			)
+		)
+		(pin "TERM_SIG" output
+			(at 232.41 63.5 180)
 			(effects
 				(font

Commit message: 🤪
Parts:
- added D3: LOGGING, symbol Device:LED
- added R10: 10 KΩ, symbol Device:R_US
- added R12: 220 Ω, symbol Device:R_US
- added R9: 4.7 KΩ, symbol Device:R_US
Connections:
- net BOOT: now also A1.5 (GPIO3)
- net GND: now also D3.1 (K), R10.1
- net GUN_FIRED: now also A1.26 (GPIO20); no longer A1.16 (GPIO12)
- net RS485_RX: now also R10.2, R9.1; no longer U3.1 (RO)
- net LOGGING: now reaches A1.27 (GPIO21)
- net LOGGING: now also R12.2
- new net: R9.2, U3.1 (RO)
- new net: D3.2 (A), R12.1
- no-connect marks 22 -> 19
