File: react_schematics/power_and_connectors.kicad_sch (KiCad schematic)
At the start: 11 parts, among them J1 Input Jack, J2 Output Jack, U1 MPM3610, U5 AQY212EHA

Commit message: new sch changes
Connections:
- net TERM_SIG: now reaches R7.2
- net ABORT_SIG renamed ABORT_SIG_IN
- net ABORT_SIG_IN: no longer J2.5
- new net ABORT_SIG_OUT: J2.5
Changed lines of the file:
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@@
-	)
-	(junction
-		(at 76.2 67.31)
-		(diameter 0)
-		(color 0 0 0 0)
 	)
 	(junction
@@
 	(wire
 		(pts
-			(xy 48.26 49.53) (xy 48.26 67.31)
-		)
-		(stroke
-			(width 0)
-			(type default)
-		)
-	)
-	(wire
-		(pts
 			(xy 58.42 55.88) (xy 76.2 55.88)
 		)
@@
 	(wire
 		(pts
+			(xy 48.26 96.52) (xy 48.26 49.53)
+		)
+		(stroke
+			(width 0)
+			(type default)
+		)
+	)
+	(wire
+		(pts
+			(xy 36.83 96.52) (xy 48.26 96.52)
+		)
+		(stroke
+			(width 0)
+			(type default)
+		)
+	)
+	(wire
+		(pts
 			(xy 76.2 72.39) (xy 106.68 72.39)
 		)
@@
 	(wire
 		(pts
+			(xy 52.07 143.51) (xy 69.85 143.51)
+		)
+		(stroke
+			(width 0)
+			(type default)
+		)
+	)
+	(wire
+		(pts
 			(xy 203.2 52.07) (xy 190.5 52.07)
 		)
@@
 	(wire
 		(pts
-			(xy 76.2 67.31) (xy 104.14 67.31)
-		)
-		(stroke
-			(width 0)
-			(type default)
-		)
-	)
-	(wire
-		(pts
 			(xy 76.2 77.47) (xy 90.17 77.47)
 		)
@@
 	(wire
 		(pts
+			(xy 114.3 96.52) (xy 104.14 96.52)
+		)
+		(stroke
+			(width 0)
+			(type default)
+		)
+	)
+	(wire
+		(pts
 			(xy 190.5 24.13) (xy 190.5 29.21)
 		)
@@
 	(wire
 		(pts
-			(xy 48.26 67.31) (xy 76.2 67.31)
-		)
-		(stroke
-			(width 0)
-			(type default)
-		)
-	)
-	(wire
-		(pts
 			(xy 90.17 77.47) (xy 90.17 92.71)
 		)
@@
 	(wire
 		(pts
+			(xy 104.14 96.52) (xy 104.14 49.53)
+		)
+		(stroke
+			(width 0)
+			(type default)
+		)
+	)
+	(wire
+		(pts
 			(xy 76.2 55.88) (xy 93.98 55.88)
 		)
@@
 	(wire
 		(pts
-			(xy 104.14 67.31) (xy 104.14 49.53)
-		)
-		(stroke
-			(width 0)
-			(type default)
-		)
-	)
-	(wire
-		(pts
-			(xy 76.2 67.31) (xy 76.2 69.85)
-		)
-		(stroke
-			(width 0)
-			(type default)
-		)
-	)
-	(wire
-		(pts
 			(xy 106.68 72.39) (xy 106.68 49.53)
 		)
@@
 		(pts
 			(xy 53.34 49.53) (xy 53.34 58.42)
-		)
-		(stroke
-			(width 0)
-			(type default)
-		)
-	)
-	(wire
-		(pts
-			(xy 76.2 69.85) (xy 77.47 69.85)
 		)
 		(stroke
@@
 				(size 1.27 1.27)
 			)
-			(justify left bottom)
+			(justify bottom)
 		)
 	)
@@
 				(size 1.27 1.27)
 			)
-			(justify left bottom)
+			(justify bottom)
+		)
+	)
+	(hierarchical_label "ABORT_SIG_IN"
+		(shape output)
+		(at 36.83 96.52 180)
+		(effects
+			(font
+				(size 1.27 1.27)
+			)
+			(justify right)
+		)
+	)
+	(hierarchical_label "ABORT_SIG_OUT"
+		(shape output)
+		(at 114.3 96.52 0)
+		(effects
+			(font
+				(size 1.27 1.27)
+			)
+			(justify left)
 		)
 	)
@@
 		)
 	)
+	(hierarchical_label "TERM_SIG"
+		(shape output)
+		(at 52.07 143.51 180)
+		(effects
+			(font
+				(size 1.27 1.27)
+			)
+			(justify right)
+		)
+	)
 	(hierarchical_label "FS_ALERT"
 		(shape bidirectional)
@@
 		(effects
 			(font
-				(size 1.27 1.27)
-			)
-			(justify left)
-		)
-	)
-	(hierarchical_label "ABORT_SIG"
-		(shape bidirectional)
-		(at 77.47 69.85 0)
-		(effects
-			(font
